Commit message: Auto stash before rebase of "master" onto "origin/master"

File: ode_bringup/model/omoda.urdf (robot description, URDF)
Before this commit: robot omoda, 8 links, 7 joints
Links:
- removed link camera
- added link camerakanan
- added link camerakiri
- added link cameratengah
Joints:
- removed joint camera_joint
- added joint camerakanan_joint: type fixed, parent base_lidar, child camerakanan, origin xyz=0.240546 -0.2273 0.19 rpy=0.0 0.0 -0.959931089
- added joint camerakiri_joint: type fixed, parent base_lidar, child camerakiri, origin xyz=0.240546 0.2273 0.19 rpy=0.0 0.0 0.959931089
- added joint cameratengah_joint: type fixed, parent base_lidar, child cameratengah, origin xyz=0.3585 0.0 0.19 rpy=0.0 0.0 0.0

Commit message: add akeh features

File: ode_bringup/model/omoda.urdf (robot description, URDF)
Before this commit: robot omoda, 10 links, 9 joints
Links:
- added link cameracalib
Joints:
- added joint cameracalib_joint: type fixed, parent lidartengah, child cameracalib, origin xyz=0.57446866 -0.08339404 -1.0530726 rpy=0.75612054 -1.02291871  0.89599662
- joint cameratengah_joint: origin xyz=0.3585 0.0 0.19 rpy=0.0 0.0 0.0 -> xyz=0.4685 -0.093 0.61 rpy=0.0 -0.07  -0.01195

Commit message: filtering flat on projected cloud

File: ode_bringup/model/omoda.urdf (robot description, URDF)
Before this commit: robot omoda, 11 links, 10 joints
Joints:
- joint cameratengah_joint: origin xyz=0.4685 -0.093 0.61 rpy=0.0 -0.07  -0.01195 -> xyz=0.4685 -0.093 0.18 rpy=0.0 -0.07  -0.01195

Commit message: change

File: ode_bringup/model/omoda.urdf (robot description, URDF)
Before this commit: robot omoda, 11 links, 10 joints
Links:
- removed link cameracalib
Joints:
- removed joint cameracalib_joint
